File: pcb/keyboard.kicad_pcb (KiCad board)
At the start: 2 copper layers, 67.9 x 97.3 mm, 41 parts, among them J1 Conn_01x04_Pin, SW1 SW_Push, SW2 SW_Push, SW3 SW_Push, SW4 SW_Push, SW5 SW_Push, SW6 SW_Push, SW7 SW_Push, SW8 SW_Push, SW9 RotaryEncoder_Switch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

Commit message: new pcb image
Other:
- board text added: "OLED SCREEN HERE"
Changed lines of the file:
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@@
+		)
+	)
+	(gr_text "OLED SCREEN HERE"
+		(at 41.068636 58.66948 0)
+		(layer "F.SilkS")
+		(effects
+			(font
+				(size 1 1)
+				(thickness 0.1)
+			)
+			(justify left bottom)
 		)
 	)
